File: ft234/ft234.kicad_pcb (KiCad board)
At the start: 2 copper layers, 14.2 x 10.2 mm, 12 parts, among them J1 USB_OTG, J2 Conn_01x04, U1 FT234XD

Commit message: update
Parts:
- added R5: 120, Resistors_SMD:R_0402_NoSilk, F.Cu at (147.6, 71.1)
- moved R3 0.82 mm to (149.9, 71.1)
Connections:
- J1 pad 4: Net-(J1-Pad4) -> (no net)
- U1 pad 10: /Rx -> Net-(R5-Pad2)
- U1 pad 8: Net-(U1-Pad8) -> (no net)
Routing:
- net Net-(R5-Pad2): track 0.00 -> 3.07 mm
- net Net-(R3-Pad2): track 3.95 -> 3.26 mm
- net /Tx: track 7.12 -> 6.45 mm
Changed lines of the file:
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@@
   (thickness 1.6)
   (drawings 22)
-  (tracks 99)
+  (tracks 101)
   (zones 0)
-  (modules 12)
-  (nets 15)
+  (modules 13)
+  (nets 14)
 )
 (page A4)
@@
 (net 11 /Rx)
 (net 12 /Tx)
-(net 13 "Net-(J1-Pad4)")
-(net 14 "Net-(U1-Pad8)")
+(net 13 "Net-(R5-Pad2)")
 (net_class Default "This is the default net class."
   (clearance 0.15)
@@
   (add_net "Net-(C2-Pad1)")
   (add_net "Net-(D1-Pad1)")
-  (add_net "Net-(J1-Pad4)")
   (add_net "Net-(R1-Pad1)")
   (add_net "Net-(R2-Pad1)")
   (add_net "Net-(R3-Pad2)")
   (add_net "Net-(R4-Pad2)")
-  (add_net "Net-(U1-Pad8)")
+  (add_net "Net-(R5-Pad2)")
 )
   (module Capacitors_SMD:C_0402_NoSilk (layer F.Cu)
@@
     (pad 3 smd rect (at -2 0.0009) (size 1.65 0.4) (layers F.Cu F.Paste F.Mask)
       (net 3 "Net-(C2-Pad1)"))
-    (pad 4 smd rect (at -2 -0.65) (size 1.65 0.4) (layers F.Cu F.Paste F.Mask)
-      (net 13 "Net-(J1-Pad4)"))
+    (pad 4 smd rect (at -2 -0.65) (size 1.65 0.4) (layers F.Cu F.Paste F.Mask))
     (pad 5 smd rect (at -2 -1.3) (size 1.65 0.4) (layers F.Cu F.Paste F.Mask)
       (net 1 GND))
@@
   )
   (module Resistors_SMD:R_0402_NoSilk (layer F.Cu)
-    (at 149.1 71.3)
+    (at 149.9 71.1)
     (descr "Resistor SMD 0402, reflow soldering, Vishay (see dcrcw.pdf)")
     (tags "resistor 0402")
@@
     (pad 7 smd rect (at 1.4 1.125 90) (size 0.7 0.25) (layers F.Cu F.Paste F.Mask)
       (net 9 "Net-(R3-Pad2)"))
-    (pad 8 smd rect (at 1.4 0.675 90) (size 0.7 0.25) (layers F.Cu F.Paste F.Mask)
-      (net 14 "Net-(U1-Pad8)"))
+    (pad 8 smd rect (at 1.4 0.675 90) (size 0.7 0.25) (layers F.Cu F.Paste F.Mask))
     (pad 9 smd rect (at 1.4 0.225 90) (size 0.7 0.25) (layers F.Cu F.Paste F.Mask)
       (net 4 +3V3))
     (pad 10 smd rect (at 1.4 -0.225 90) (size 0.7 0.25) (layers F.Cu F.Paste F.Mask)
-      (net 11 /Rx))
+      (net 13 "Net-(R5-Pad2)"))
     (pad 11 smd rect (at 1.4 -0.675 90) (size 0.7 0.25) (layers F.Cu F.Paste F.Mask)
       (net 1 GND))
@@
     )
   )
+  (module Resistors_SMD:R_0402_NoSilk (layer F.Cu)
+    (at 147.6 71.1)
+    (descr "Resistor SMD 0402, reflow soldering, Vishay (see dcrcw.pdf)")
+    (tags "resistor 0402")
+    (attr smd)
+    (fp_text reference R5 (at 0 -1.2) (layer F.SilkS)
+      (effects (font (size 1 1) (thickness 0.15)))
+    )
+    (fp_text value 120 (at 0 1.25) (layer F.Fab)
+      (effects (font (size 1 1) (thickness 0.15)))
+    )
+    (fp_text user %R (at 0 -1.2) (layer F.Fab)
+      (effects (font (size 1 1) (thickness 0.15)))
+    )
+    (fp_line (start -0.5 0.25) (end -0.5 -0.25) (layer F.Fab) (width 0.1))
+    (fp_line (start 0.5 0.25) (end -0.5 0.25) (layer F.Fab) (width 0.1))
+    (fp_line (start 0.5 -0.25) (end 0.5 0.25) (layer F.Fab) (width 0.1))
+    (fp_line (start -0.5 -0.25) (end 0.5 -0.25) (layer F.Fab) (width 0.1))
+    (fp_line (start -0.8 -0.45) (end 0.8 -0.45) (layer F.CrtYd) (width 0.05))
+    (fp_line (start -0.8 -0.45) (end -0.8 0.45) (layer F.CrtYd) (width 0.05))
+    (fp_line (start 0.8 0.45) (end 0.8 -0.45) (layer F.CrtYd) (width 0.05))
+    (fp_line (start 0.8 0.45) (end -0.8 0.45) (layer F.CrtYd) (width 0.05))
+    (pad 1 smd rect (at -0.45 0) (size 0.4 0.6) (layers F.Cu F.Paste F.Mask)
+      (net 11 /Rx))
+    (pad 2 smd rect (at 0.45 0) (size 0.4 0.6) (layers F.Cu F.Paste F.Mask)
+      (net 13 "Net-(R5-Pad2)"))
+    (model ${KISYS3DMOD}/Resistors_SMD.3dshapes/R_0402.wrl
+      (at (xyz 0 0 0))
+      (scale (xyz 1 1 1))
+      (rotate (xyz 0 0 0))
+    )
+  )
   (gr_text FT234 (at 143 75) (layer B.Mask)
     (effects (font (size 1.2 1.2) (thickness 0.25)) (justify mirror))
@@
   (gr_line (start 150.5 73.7) (end 150.7 73.8) (layer B.Mask) (width 0.2))
   (gr_line (start 150.4 74.4) (end 150.4 73.4) (layer B.Mask) (width 0.2))
-  (gr_line (start 149.3 71.3) (end 149.1 71.2) (layer B.Mask) (width 0.2))
-  (gr_line (start 149.1 70.9) (end 149.3 71.3) (layer B.Mask) (width 0.2))
-  (gr_line (start 149.4 70.9) (end 149.1 70.9) (layer B.Mask) (width 0.2))
-  (gr_line (start 149.4 71.6) (end 148.8 71.1) (layer B.Mask) (width 0.2))
-  (gr_line (start 149.4 70.6) (end 149.4 71.6) (layer B.Mask) (width 0.2))
-  (gr_line (start 148.8 71.1) (end 149.4 70.6) (layer B.Mask) (width 0.2))
-  (gr_line (start 150.9 71.1) (end 149.1 71.1) (layer B.Mask) (width 0.4))
+  (gr_line (start 149.9 71) (end 149.7 70.9) (layer B.Mask) (width 0.2))
+  (gr_line (start 149.7 70.6) (end 149.9 71) (layer B.Mask) (width 0.2))
+  (gr_line (start 150 70.6) (end 149.7 70.6) (layer B.Mask) (width 0.2))
+  (gr_line (start 150 71.3) (end 149.4 70.8) (layer B.Mask) (width 0.2))
+  (gr_line (start 150 70.3) (end 150 71.3) (layer B.Mask) (width 0.2))
+  (gr_line (start 149.4 70.8) (end 150 70.3) (layer B.Mask) (width 0.2))
+  (gr_line (start 151.5 70.8) (end 149.7 70.8) (layer B.Mask) (width 0.4))
   (gr_line (start 140 80.2) (end 140 70) (layer Edge.Cuts) (width 0.15))
   (gr_line (start 154.2 80.2) (end 140 80.2) (layer Edge.Cuts) (width 0.15))
@@
   (segment (start 147.9 73.5) (end 147.75 73.65) (width 0.15) (layer F.Cu) (net 8))
   (segment (start 147.75 73.65) (end 147.3 73.65) (width 0.15) (layer F.Cu) (net 8))
-  (segment (start 150.5 71.3) (end 149.55 71.3) (width 0.2) (layer F.Cu) (net 9))
-  (segment (start 151.2 72) (end 150.5 71.3) (width 0.2) (layer F.Cu) (net 9))
-  (segment (start 151.2 73.05) (end 151.2 72) (width 0.2) (layer F.Cu) (net 9))
+  (segment (start 151.2 73.05) (end 151.2 72.05) (width 0.2) (layer F.Cu) (net 9))
+  (segment (start 151.2 72.05) (end 150.35 71.2) (width 0.2) (layer F.Cu) (net 9))
+  (segment (start 150.35 71.2) (end 150.35 71.1) (width 0.2) (layer F.Cu) (net 9))
   (segment (start 150.425 73.5) (end 150.75 73.5) (width 0.2) (layer F.Cu) (net 9))
   (segment (start 150.75 73.5) (end 151.2 73.05) (width 0.2) (layer F.Cu) (net 9))
@@
   (segment (start 151.300001 78.449999) (end 150.85 78.9) (width 0.2) (layer F.Cu) (net 10))
   (segment (start 150.85 78.9) (end 150.85 79) (width 0.2) (layer F.Cu) (net 10))
-  (segment (start 149.1 72.925) (end 149.075 72.95) (width 0.19) (layer F.Cu) (net 11))
-  (segment (start 149.075 72.95) (end 149.075 73.5) (width 0.19) (layer F.Cu) (net 11))
-  (segment (start 149.2 70.7) (end 151.25 70.7) (width 0.2) (layer F.Cu) (net 11))
-  (segment (start 151.25 70.7) (end 151.85 71.3) (width 0.2) (layer F.Cu) (net 11))
-  (segment (start 151.85 71.3) (end 152.9 71.3) (width 0.2) (layer F.Cu) (net 11))
-  (segment (start 149.1 70.8) (end 149.2 70.7) (width 0.2) (layer F.Cu) (net 11))
-  (segment (start 149.1 72.925) (end 149.1 70.8) (width 0.19) (layer F.Cu) (net 11))
+  (segment (start 147.600001 70.549999) (end 150.849999 70.549999) (width 0.2) (layer F.Cu) (net 11))
+  (segment (start 147.15 71) (end 147.600001 70.549999) (width 0.2) (layer F.Cu) (net 11))
+  (segment (start 150.849999 70.549999) (end 151.6 71.3) (width 0.2) (layer F.Cu) (net 11))
+  (segment (start 151.6 71.3) (end 152.9 71.3) (width 0.2) (layer F.Cu) (net 11))
+  (segment (start 147.15 71.1) (end 147.15 71) (width 0.2) (layer F.Cu) (net 11))
   (segment (start 152.45 70.85) (end 152.9 71.3) (width 0.15) (layer F.Cu) (net 11))
-  (segment (start 152.9 73.84) (end 151.3 72.24) (width 0.2) (layer B.Cu) (net 12))
-  (segment (start 148.8 72.1) (end 148 71.3) (width 0.2) (layer B.Cu) (net 12))
-  (segment (start 151.3 72.24) (end 151.3 72) (width 0.2) (layer B.Cu) (net 12))
-  (segment (start 151.3 72) (end 150.950002 71.650002) (width 0.2) (layer B.Cu) (net 12))
-  (segment (start 150.950002 71.650002) (end 150.049998 71.650002) (width 0.2) (layer B.Cu) (net 12))
-  (segment (start 150.049998 71.650002) (end 149.6 72.1) (width 0.2) (layer B.Cu) (net 12))
-  (segment (start 149.6 72.1) (end 148.8 72.1) (width 0.2) (layer B.Cu) (net 12))
-  (segment (start 148.65 71.3) (end 148 71.3) (width 0.2) (layer F.Cu) (net 12))
-  (via (at 148 71.3) (size 0.6) (drill 0.3) (layers F.Cu B.Cu) (net 12))
+  (segment (start 148.9 71.1) (end 149.5 71.7) (width 0.2) (layer B.Cu) (net 12))
+  (segment (start 149.5 71.7) (end 150.8 71.7) (width 0.2) (layer B.Cu) (net 12))
+  (segment (start 150.8 71.7) (end 151.2 72.1) (width 0.2) (layer B.Cu) (net 12))
+  (segment (start 151.2 72.1) (end 151.2 73.4) (width 0.2) (layer B.Cu) (net 12))
+  (segment (start 151.2 73.4) (end 151.64 73.84) (width 0.2) (layer B.Cu) (net 12))
+  (segment (start 151.64 73.84) (end 152.9 73.84) (width 0.2) (layer B.Cu) (net 12))
+  (segment (start 149.45 71.1) (end 148.9 71.1) (width 0.2) (layer F.Cu) (net 12))
+  (via (at 148.9 71.1) (size 0.6) (drill 0.3) (layers F.Cu B.Cu) (net 12))
+  (segment (start 148.524999 71.674999) (end 148.05 71.2) (width 0.2) (layer F.Cu) (net 13))
+  (segment (start 148.950001 71.674999) (end 148.524999 71.674999) (width 0.2) (layer F.Cu) (net 13))
+  (segment (start 149.075 73.5) (end 149.075 71.799998) (width 0.2) (layer F.Cu) (net 13))
+  (segment (start 149.075 71.799998) (end 148.950001 71.674999) (width 0.2) (layer F.Cu) (net 13))
+  (segment (start 148.05 71.2) (end 148.05 71.1) (width 0.2) (layer F.Cu) (net 13))
   (zone (net 1) (net_name GND) (layer F.Cu) (hatch edge 0.508)
     (connect_pads yes (clearance 0.15))
