File: ft234/ft234.sch (KiCad schematic (older format))
At the start: 12 parts, among them J1 USB_OTG, J2 Conn_01x04, U1 FT234XD

Commit message: update
Parts:
- added R5: 120, Resistors_SMD:R_0402_NoSilk, symbol R
Connections:
- net Rx: now also R5.1; no longer U1.10 (RXD)
- new net: R5.2, U1.10 (RXD)
Other:
- moved on the sheet: J2
Changed lines of the file:
@@
 L Conn_01x04 J2
 U 1 1 59CBBCFF
-P 6950 3350
-F 0 "J2" H 7050 3450 50  0000 L CNN
-F 1 "Conn_01x04" H 6900 3550 50  0000 L CNN
-F 2 "Pin_Headers:Pin_Header_Straight_1x04_Pitch2.54mm" H 6950 3350 50  0001 C CNN
-F 3 "" H 6950 3350 50  0001 C CNN
-	1    6950 3350
+P 7600 3350
+F 0 "J2" H 7700 3450 50  0000 L CNN
+F 1 "Conn_01x04" H 7550 3550 50  0000 L CNN
+F 2 "Pin_Headers:Pin_Header_Straight_1x04_Pitch2.54mm" H 7600 3350 50  0001 C CNN
+F 3 "" H 7600 3350 50  0001 C CNN
+	1    7600 3350
 	1    0    0    -1
 $EndComp
@@
 L GND #PWR02
 U 1 1 59CBBDF1
-P 6400 3450
-F 0 "#PWR02" H 6400 3200 50  0001 C CNN
-F 1 "GND" H 6405 3277 50  0000 C CNN
-F 2 "" H 6400 3450 50  0001 C CNN
-F 3 "" H 6400 3450 50  0001 C CNN
-	1    6400 3450
+P 7050 3450
+F 0 "#PWR02" H 7050 3200 50  0001 C CNN
+F 1 "GND" H 7055 3277 50  0000 C CNN
+F 2 "" H 7050 3450 50  0001 C CNN
+F 3 "" H 7050 3450 50  0001 C CNN
+	1    7050 3450
 	1    0    0    -1
 $EndComp
@@
 L +3V3 #PWR03
 U 1 1 59CBBEC4
-P 7100 3650
-F 0 "#PWR03" H 7100 3500 50  0001 C CNN
-F 1 "+3V3" H 7115 3823 50  0000 C CNN
-F 2 "" H 7100 3650 50  0001 C CNN
-F 3 "" H 7100 3650 50  0001 C CNN
-	1    7100 3650
+P 7750 3650
+F 0 "#PWR03" H 7750 3500 50  0001 C CNN
+F 1 "+3V3" H 7765 3823 50  0000 C CNN
+F 2 "" H 7750 3650 50  0001 C CNN
+F 3 "" H 7750 3650 50  0001 C CNN
+	1    7750 3650
 	1    0    0    -1
 $EndComp
@@
 	4500 3000 4850 3000
 Wire Wire Line
-	6750 3650 6750 3550
-Wire Wire Line
-	7100 3650 6750 3650
-Wire Wire Line
-	6750 3450 6400 3450
+	7400 3650 7400 3550
+Wire Wire Line
+	7750 3650 7400 3650
+Wire Wire Line
+	7400 3450 7050 3450
 Wire Wire Line
 	6250 3500 6000 3500
@@
 	6100 3700 6000 3700
 Wire Wire Line
-	6750 3350 6450 3350
-Wire Wire Line
-	6450 3350 6450 3100
-Wire Wire Line
-	6750 3250 6250 3250
+	7400 3350 7100 3350
+Wire Wire Line
+	7100 3100 6450 3100
+Wire Wire Line
+	7400 3250 6750 3250
 Wire Wire Line
 	6250 3250 6250 3500
-Text Label 6750 3350 2    60   ~ 0
+Text Label 7400 3350 2    60   ~ 0
 Tx
-Text Label 6750 3250 2    60   ~ 0
+Text Label 7400 3250 2    60   ~ 0
 Rx
 Wire Wire Line
@@
 Wire Wire Line
 	6000 4050 6050 4050
+Wire Wire Line
+	7100 3350 7100 3100
+$Comp
+L R R5
+U 1 1 59F30B2F
+P 6600 3250
+F 0 "R5" V 6500 3250 50  0000 C CNN
+F 1 "120" V 6600 3250 50  0000 C CNN
+F 2 "Resistors_SMD:R_0402_NoSilk" V 6530 3250 50  0001 C CNN
+F 3 "" H 6600 3250 50  0001 C CNN
+	1    6600 3250
+	0    1    1    0
+$EndComp
+Wire Wire Line
+	6250 3250 6450 3250
 $EndSCHEMATC

Commit message: hmm
Parts:
- C1, C2, C3, C4: symbol C -> ft234-rescue:C
- D1: symbol LED -> ft234-rescue:LED
- J1: symbol USB_OTG -> ft234-rescue:USB_OTG
- J2: symbol Conn_01x04 -> ft234-rescue:Conn_01x04
- R1, R2, R3, R4, R5: symbol R -> ft234-rescue:R
- U1: symbol FT234XD -> ft234xd:FT234XD
Changed lines of the file:
@@
-EESchema Schematic File Version 3
-LIBS:power
-LIBS:device
-LIBS:linear
-LIBS:regul
-LIBS:adc-dac
-LIBS:memory
-LIBS:xilinx
-LIBS:microcontrollers
-LIBS:dsp
-LIBS:microchip
-LIBS:analog_switches
-LIBS:motorola
-LIBS:texas
-LIBS:intel
-LIBS:audio
-LIBS:interface
-LIBS:digital-audio
-LIBS:philips
-LIBS:cypress
-LIBS:siliconi
-LIBS:opto
-LIBS:atmel
-LIBS:contrib
-LIBS:ft234xd
-LIBS:ft230-cache
+EESchema Schematic File Version 4
 LIBS:ft234-cache
-EELAYER 26 0
+EELAYER 29 0
 EELAYER END
 $Descr A4 11693 8268
@@
 $EndDescr
 $Comp
-L GND #PWR01
+L power:GND #PWR01
 U 1 1 59CBBAFA
 P 5400 4200
@@
 $EndComp
 $Comp
-L R R3
+L ft234-rescue:R R3
 U 1 1 59CBBB72
 P 6300 3100
@@
 $EndComp
 $Comp
-L Conn_01x04 J2
+L ft234-rescue:Conn_01x04 J2
 U 1 1 59CBBCFF
 P 7600 3350
@@
 $EndComp
 $Comp
-L GND #PWR02
+L power:GND #PWR02
 U 1 1 59CBBDF1
 P 7050 3450
@@
 $EndComp
 $Comp
-L +3V3 #PWR03
+L power:+3V3 #PWR03
 U 1 1 59CBBEC4
 P 7750 3650
@@
 $EndComp
 $Comp
-L +3V3 #PWR04
+L power:+3V3 #PWR04
 U 1 1 59CBBF9A
 P 4500 3000
@@
 $EndComp
 $Comp
-L R R4
+L ft234-rescue:R R4
 U 1 1 59CBC039
 P 6200 4050
@@
 $EndComp
 $Comp
-L C C3
+L ft234-rescue:C C3
 U 1 1 59CBC175
 P 4500 3150
@@
 $EndComp
 $Comp
-L GND #PWR05
+L power:GND #PWR05
 U 1 1 59CBC250
 P 4500 3300
@@
 $EndComp
 $Comp
-L R R1
+L ft234-rescue:R R1
 U 1 1 59CBC267
 P 4050 3550
@@
 $EndComp
 $Comp
-L R R2
+L ft234-rescue:R R2
 U 1 1 59CBC2E6
 P 4050 3750
@@
 $EndComp
 $Comp
-L C C2
+L ft234-rescue:C C2
 U 1 1 59CBC39F
 P 3900 4000
@@
 $EndComp
 $Comp
-L C C1
+L ft234-rescue:C C1
 U 1 1 59CBC4AC
 P 3650 4000
@@
 $EndComp
 $Comp
-L GND #PWR06
+L power:GND #PWR06
 U 1 1 59CBC538
 P 3900 4250
@@
 $EndComp
 $Comp
-L LED D1
+L ft234-rescue:LED D1
 U 1 1 59CBC8A8
 P 6650 4050
@@
 $EndComp
 $Comp
-L +3V3 #PWR07
+L power:+3V3 #PWR07
 U 1 1 59CBCA7C
 P 6900 4050
@@
 $EndComp
 $Comp
-L +3V3 #PWR08
+L power:+3V3 #PWR08
 U 1 1 59CBCC93
 P 4550 3950
@@
 $EndComp
 $Comp
-L +3V3 #PWR09
+L power:+3V3 #PWR09
 U 1 1 59CBCCED
 P 5600 3050
@@
 $EndComp
 $Comp
-L C C4
+L ft234-rescue:C C4
 U 1 1 59CBCDB8
 P 5200 2750
@@
 $EndComp
 $Comp
-L GND #PWR010
+L power:GND #PWR010
 U 1 1 59CBCEAD
 P 5200 2900
@@
 $EndComp
 $Comp
-L +5V #PWR011
+L power:+5V #PWR011
 U 1 1 59CBCF7B
 P 5200 2500
@@
 $EndComp
 $Comp
-L USB_OTG J1
+L ft234-rescue:USB_OTG J1
 U 1 1 59CBD396
 P 2900 3600
@@
 $EndComp
 $Comp
-L +5V #PWR012
+L power:+5V #PWR012
 U 1 1 59CBD416
 P 3350 3400
@@
 $EndComp
 $Comp
-L GND #PWR013
+L power:GND #PWR013
 U 1 1 59CBD672
 P 2900 4100
@@
 	3650 3550 3650 3850
 Wire Wire Line
-	3350 3550 3900 3550
+	3350 3550 3650 3550
 Wire Wire Line
 	3900 3750 3900 3850
@@
 	5500 4200 5500 4100
 $Comp
-L GND #PWR014
+L power:GND #PWR014
 U 1 1 59CBDE8C
 P 6200 3650
@@
 	5400 4200 5500 4200
 $Comp
-L FT234XD U1
+L ft234xd:FT234XD U1
 U 1 1 59EF5B28
 P 5450 3600
@@
 	7100 3350 7100 3100
 $Comp
-L R R5
+L ft234-rescue:R R5
 U 1 1 59F30B2F
 P 6600 3250
@@
 Wire Wire Line
 	6250 3250 6450 3250
+Wire Wire Line
+	3650 3550 3900 3550
 $EndSCHEMATC
