File: ft230/ft230.sch (KiCad schematic (older format))
At the start: 14 parts, among them J1 USB_OTG, J2 Conn_01x04, U1 FT230XQ

Commit message: exchange Rx and Tx
Connections:
- net Rx: now reaches U1.2 (RXD)
- net Rx: now also J2.1 (Pin_1); no longer J2.2 (Pin_2)
- net Tx: now reaches R3.1
- net Tx: now also J2.2 (Pin_2); no longer J2.1 (Pin_1)
Other:
- moved on the sheet: R3
Changed lines of the file:
@@
 LIBS:power
 LIBS:device
-LIBS:transistors
-LIBS:conn
 LIBS:linear
 LIBS:regul
-LIBS:74xx
-LIBS:cmos4000
 LIBS:adc-dac
 LIBS:memory
@@
 LIBS:digital-audio
 LIBS:philips
-LIBS:display
 LIBS:cypress
 LIBS:siliconi
@@
 LIBS:atmel
 LIBS:contrib
-LIBS:valves
 LIBS:ft230xq
+LIBS:ft230-cache
 EELAYER 26 0
 EELAYER END
@@
 L R R3
 U 1 1 59CBBB72
-P 6300 3100
-F 0 "R3" V 6200 3100 50  0000 C CNN
-F 1 "120" V 6300 3100 50  0000 C CNN
-F 2 "Resistors_SMD:R_0402_NoSilk" V 6230 3100 50  0001 C CNN
-F 3 "" H 6300 3100 50  0001 C CNN
-	1    6300 3100
+P 6300 2950
+F 0 "R3" V 6200 2950 50  0000 C CNN
+F 1 "120" V 6300 2950 50  0000 C CNN
+F 2 "Resistors_SMD:R_0402_NoSilk" V 6230 2950 50  0001 C CNN
+F 3 "" H 6300 2950 50  0001 C CNN
+	1    6300 2950
 	0    1    1    0
 $EndComp
@@
 	6750 3300 6400 3300
 Wire Wire Line
-	6250 3200 6750 3200
-Wire Wire Line
-	6250 3350 6250 3200
-Wire Wire Line
-	6000 3350 6250 3350
-Wire Wire Line
-	6450 3100 6750 3100
+	6250 3350 6000 3350
 Wire Wire Line
 	6150 3250 6000 3250
 Wire Wire Line
-	6150 3100 6150 3250
+	6150 2950 6150 3250
 Wire Wire Line
 	5400 4300 5400 4200
@@
 Wire Wire Line
 	6100 3550 6000 3550
+Wire Wire Line
+	6750 3200 6450 3200
+Wire Wire Line
+	6450 3200 6450 2950
+Wire Wire Line
+	6750 3100 6250 3100
+Wire Wire Line
+	6250 3100 6250 3350
+Text Label 6750 3200 2    60   ~ 0
+Tx
+Text Label 6750 3100 2    60   ~ 0
+Rx
 $EndSCHEMATC

Commit message: update
Parts:
- added R6: 120, Resistors_SMD:R_0402_NoSilk, symbol R
Connections:
- net Rx: now also R6.1; no longer U1.2 (RXD)
- new net: R6.2, U1.2 (RXD)
Other:
- moved on the sheet: J2
Changed lines of the file:
@@
 L Conn_01x04 J2
 U 1 1 59CBBCFF
-P 6950 3200
-F 0 "J2" H 7050 3300 50  0000 L CNN
-F 1 "Conn_01x04" H 6900 3400 50  0000 L CNN
-F 2 "Pin_Headers:Pin_Header_Straight_1x04_Pitch2.54mm" H 6950 3200 50  0001 C CNN
-F 3 "" H 6950 3200 50  0001 C CNN
-	1    6950 3200
+P 7500 3200
+F 0 "J2" H 7600 3300 50  0000 L CNN
+F 1 "Conn_01x04" H 7450 3400 50  0000 L CNN
+F 2 "Pin_Headers:Pin_Header_Straight_1x04_Pitch2.54mm" H 7500 3200 50  0001 C CNN
+F 3 "" H 7500 3200 50  0001 C CNN
+	1    7500 3200
 	1    0    0    -1
 $EndComp
@@
 L GND #PWR02
 U 1 1 59CBBDF1
-P 6400 3300
-F 0 "#PWR02" H 6400 3050 50  0001 C CNN
-F 1 "GND" H 6405 3127 50  0000 C CNN
-F 2 "" H 6400 3300 50  0001 C CNN
-F 3 "" H 6400 3300 50  0001 C CNN
-	1    6400 3300
+P 7150 3300
+F 0 "#PWR02" H 7150 3050 50  0001 C CNN
+F 1 "GND" H 7155 3127 50  0000 C CNN
+F 2 "" H 7150 3300 50  0001 C CNN
+F 3 "" H 7150 3300 50  0001 C CNN
+	1    7150 3300
 	1    0    0    -1
 $EndComp
@@
 L +3V3 #PWR03
 U 1 1 59CBBEC4
-P 7100 3500
-F 0 "#PWR03" H 7100 3350 50  0001 C CNN
-F 1 "+3V3" H 7115 3673 50  0000 C CNN
-F 2 "" H 7100 3500 50  0001 C CNN
-F 3 "" H 7100 3500 50  0001 C CNN
-	1    7100 3500
+P 7650 3500
+F 0 "#PWR03" H 7650 3350 50  0001 C CNN
+F 1 "+3V3" H 7665 3673 50  0000 C CNN
+F 2 "" H 7650 3500 50  0001 C CNN
+F 3 "" H 7650 3500 50  0001 C CNN
+	1    7650 3500
 	1    0    0    -1
 $EndComp
@@
 	4500 3000 4850 3000
 Wire Wire Line
-	6750 3500 6750 3400
-Wire Wire Line
-	7100 3500 6750 3500
-Wire Wire Line
-	6750 3300 6400 3300
+	7300 3500 7300 3400
+Wire Wire Line
+	7650 3500 7300 3500
+Wire Wire Line
+	7300 3300 7150 3300
 Wire Wire Line
 	6250 3350 6000 3350
@@
 	6100 3550 6000 3550
 Wire Wire Line
-	6750 3200 6450 3200
+	7300 3200 6450 3200
 Wire Wire Line
 	6450 3200 6450 2950
 Wire Wire Line
-	6750 3100 6250 3100
+	7300 3100 6850 3100
 Wire Wire Line
 	6250 3100 6250 3350
-Text Label 6750 3200 2    60   ~ 0
+Text Label 7300 3200 2    60   ~ 0
 Tx
-Text Label 6750 3100 2    60   ~ 0
+Text Label 7300 3100 2    60   ~ 0
 Rx
+$Comp
+L R R6
+U 1 1 59F30FB9
+P 6700 3100
+F 0 "R6" V 6600 3100 50  0000 C CNN
+F 1 "120" V 6700 3100 50  0000 C CNN
+F 2 "Resistors_SMD:R_0402_NoSilk" V 6630 3100 50  0001 C CNN
+F 3 "" H 6700 3100 50  0001 C CNN
+	1    6700 3100
+	0    1    1    0
+$EndComp
+Wire Wire Line
+	6250 3100 6550 3100
 $EndSCHEMATC

Commit message: hmm
Parts:
- C1, C2, C3, C4: symbol C -> ft230-rescue:C
- D1, D2: symbol LED -> ft230-rescue:LED
- J1: symbol USB_OTG -> ft230-rescue:USB_OTG
- J2: symbol Conn_01x04 -> ft230-rescue:Conn_01x04
- R1, R2, R3, R4, R5, R6: symbol R -> ft230-rescue:R
- U1: symbol FT230XQ -> ft230xq:FT230XQ
Changed lines of the file:
@@
-EESchema Schematic File Version 3
-LIBS:power
-LIBS:device
-LIBS:linear
-LIBS:regul
-LIBS:adc-dac
-LIBS:memory
-LIBS:xilinx
-LIBS:microcontrollers
-LIBS:dsp
-LIBS:microchip
-LIBS:analog_switches
-LIBS:motorola
-LIBS:texas
-LIBS:intel
-LIBS:audio
-LIBS:interface
-LIBS:digital-audio
-LIBS:philips
-LIBS:cypress
-LIBS:siliconi
-LIBS:opto
-LIBS:atmel
-LIBS:contrib
-LIBS:ft230xq
+EESchema Schematic File Version 4
 LIBS:ft230-cache
-EELAYER 26 0
+EELAYER 29 0
 EELAYER END
 $Descr A4 11693 8268
@@
 $EndDescr
 $Comp
-L FT230XQ U1
+L ft230xq:FT230XQ U1
 U 1 1 59CBB9E6
 P 5400 3600
@@
 $EndComp
 $Comp
-L GND #PWR01
+L power:GND #PWR01
 U 1 1 59CBBAFA
 P 5400 4300
@@
 $EndComp
 $Comp
-L R R3
+L ft230-rescue:R R3
 U 1 1 59CBBB72
 P 6300 2950
@@
 $EndComp
 $Comp
-L Conn_01x04 J2
+L ft230-rescue:Conn_01x04 J2
 U 1 1 59CBBCFF
 P 7500 3200
@@
 $EndComp
 $Comp
-L GND #PWR02
+L power:GND #PWR02
 U 1 1 59CBBDF1
 P 7150 3300
@@
 $EndComp
 $Comp
-L +3V3 #PWR03
+L power:+3V3 #PWR03
 U 1 1 59CBBEC4
 P 7650 3500
@@
 $EndComp
 $Comp
-L +3V3 #PWR04
+L power:+3V3 #PWR04
 U 1 1 59CBBF9A
 P 4500 3000
@@
 $EndComp
 $Comp
-L R R4
+L ft230-rescue:R R4
 U 1 1 59CBC039
 P 6550 3900
@@
 $EndComp
 $Comp
-L R R5
+L ft230-rescue:R R5
 U 1 1 59CBC085
 P 6550 4100
@@
 $EndComp
 $Comp
-L C C3
+L ft230-rescue:C C3
 U 1 1 59CBC175
 P 4500 3150
@@
 $EndComp
 $Comp
-L GND #PWR05
+L power:GND #PWR05
 U 1 1 59CBC250
 P 4500 3300
@@
 $EndComp
 $Comp
-L R R1
+L ft230-rescue:R R1
 U 1 1 59CBC267
 P 4050 3550
@@
 $EndComp
 $Comp
-L R R2
+L ft230-rescue:R R2
 U 1 1 59CBC2E6
 P 4050 3750
@@
 $EndComp
 $Comp
-L C C2
+L ft230-rescue:C C2
 U 1 1 59CBC39F
 P 3900 4000
@@
 $EndComp
 $Comp
-L C C1
+L ft230-rescue:C C1
 U 1 1 59CBC4AC
 P 3650 4000
@@
 $EndComp
 $Comp
-L GND #PWR06
+L power:GND #PWR06
 U 1 1 59CBC538
 P 3900 4250
@@
 $EndComp
 $Comp
-L LED D1
+L ft230-rescue:LED D1
 U 1 1 59CBC8A8
 P 7200 4050
@@
 $EndComp
 $Comp
-L LED D2
+L ft230-rescue:LED D2
 U 1 1 59CBC8FC
 P 7200 4250
@@
 $EndComp
 $Comp
-L +3V3 #PWR07
+L power:+3V3 #PWR07
 U 1 1 59CBCA7C
 P 7500 4050
@@
 $EndComp
 $Comp
-L +3V3 #PWR08
+L power:+3V3 #PWR08
 U 1 1 59CBCC93
 P 4550 3950
@@
 $EndComp
 $Comp
-L +3V3 #PWR09
+L power:+3V3 #PWR09
 U 1 1 59CBCCED
 P 5600 2950
@@
 $EndComp
 $Comp
-L C C4
+L ft230-rescue:C C4
 U 1 1 59CBCDB8
 P 5200 2650
@@
 $EndComp
 $Comp
-L GND #PWR010
+L power:GND #PWR010
 U 1 1 59CBCEAD
 P 5200 2800
@@
 $EndComp
 $Comp
-L +5V #PWR011
+L power:+5V #PWR011
 U 1 1 59CBCF7B
 P 5200 2400
@@
 $EndComp
 $Comp
-L USB_OTG J1
+L ft230-rescue:USB_OTG J1
 U 1 1 59CBD396
 P 2900 3600
@@
 $EndComp
 $Comp
-L +5V #PWR012
+L power:+5V #PWR012
 U 1 1 59CBD416
 P 3350 3400
@@
 $EndComp
 $Comp
-L GND #PWR013
+L power:GND #PWR013
 U 1 1 59CBD672
 P 2900 4100
@@
 	3650 3550 3650 3850
 Wire Wire Line
-	3350 3550 3900 3550
+	3350 3550 3650 3550
 Wire Wire Line
 	3900 3750 3900 3850
@@
 	5300 4300 5300 4200
 Wire Wire Line
-	5300 4300 5500 4300
-$Comp
-L GND #PWR014
+	5300 4300 5400 4300
+$Comp
+L power:GND #PWR014
 U 1 1 59CBDE8C
 P 6200 3500
@@
 Rx
 $Comp
-L R R6
+L ft230-rescue:R R6
 U 1 1 59F30FB9
 P 6700 3100
@@
 Wire Wire Line
 	6250 3100 6550 3100
+Wire Wire Line
+	3650 3550 3900 3550
+Wire Wire Line
+	5400 4300 5500 4300
 $EndSCHEMATC
